File: serial-breakout/serial.brd (EAGLE design)
At the start: 39.4 x 21.6 mm, 4 parts, among them X1 2510-

Commit message: label up the breakout
Connections:
- net TCK renamed LEFT
- net TDI renamed UP
- net TDO renamed RIGHT
- net TMS renamed DOWN
Changed lines of the file:
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@@
 <contactref element="X1" pad="10"/>
 </signal>
-<signal name="TDO">
+<signal name="RIGHT">
 <contactref element="X1" pad="7"/>
 </signal>
-<signal name="TDI">
+<signal name="UP">
 <contactref element="X1" pad="1"/>
 </signal>
-<signal name="TMS">
+<signal name="DOWN">
 <contactref element="X1" pad="3"/>
 </signal>
-<signal name="TCK">
+<signal name="LEFT">
 <contactref element="X1" pad="5"/>
 </signal>
