File: serial-breakout/serial.sch (EAGLE design)
At the start: 4 parts, among them X1 2510-

Commit message: label up the breakout
Connections:
- net TCK renamed LEFT
- net TDI renamed UP
- net TDO renamed RIGHT
- net TMS renamed DOWN
Other:
- note added: "FTDI 5V TTL serial"
- note added: "MIDI OUT"
- moved on the sheet: R1
Changed lines of the file:
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@@
 5
 -</text>
+<text x="127" y="157.48" size="1.778" layer="91">FTDI 5V TTL serial</text>
+<text x="127" y="193.04" size="1.778" layer="91">MIDI OUT</text>
 </plain>
 <instances>
@@
 <instance part="JP1" gate="A" x="127" y="172.72" rot="R180"/>
 <instance part="U$1" gate="G$1" x="134.62" y="208.28"/>
-<instance part="R1" gate="G$1" x="162.56" y="205.74"/>
+<instance part="R1" gate="G$1" x="157.48" y="210.82" rot="R90"/>
 </instances>
 <busses>
@@
 <pinref part="U$1" gate="G$1" pin="2"/>
 <wire x1="149.86" y1="203.2" x2="157.48" y2="203.2" width="0.1524" layer="91"/>
-<label x="157.48" y="200.66" size="1.778" layer="95" rot="R270" xref="yes"/>
+<label x="157.48" y="203.2" size="1.778" layer="95" rot="R270" xref="yes"/>
 </segment>
 </net>
@@
 <segment>
 <pinref part="R1" gate="G$1" pin="2"/>
-<wire x1="167.64" y1="205.74" x2="172.72" y2="205.74" width="0.1524" layer="91"/>
-<label x="172.72" y="205.74" size="1.778" layer="95" xref="yes"/>
+<wire x1="157.48" y1="215.9" x2="157.48" y2="218.44" width="0.1524" layer="91"/>
+<label x="157.48" y="218.44" size="1.778" layer="95" rot="R90" xref="yes"/>
 </segment>
 </net>
@@
 </segment>
 </net>
-<net name="TDO" class="0">
+<net name="RIGHT" class="0">
 <segment>
 <pinref part="X1" gate="-7" pin="KL"/>
@@
 </segment>
 </net>
-<net name="TDI" class="0">
+<net name="UP" class="0">
 <segment>
 <pinref part="X1" gate="-1" pin="KL"/>
@@
 </segment>
 </net>
-<net name="TMS" class="0">
+<net name="DOWN" class="0">
 <segment>
 <pinref part="X1" gate="-3" pin="KL"/>
@@
 </segment>
 </net>
-<net name="TCK" class="0">
+<net name="LEFT" class="0">
 <segment>
 <pinref part="X1" gate="-5" pin="KL"/>
