File: serial-breakout/super-serial.sch (EAGLE design)
At the start: 7 parts, among them X1 2510-, X2 D-SUB9-H2M09ST

Commit message: add super serial
Parts:
- added D1, D2, D3: (no value), adafruit:DIODEDO-1N4148
- added R3: 10k, rcl:R-EU_0204/7
Connections:
- new net CH_PD: D2.A, JP3.6
- new net ESP-RX: D1.A, JP3.1, R3.2
- new net RST: D3.A, JP3.4
- net 3V3: now also R3.1
- net FIRE: now also D3.C; no longer JP3.6
- net TX: now also D1.C; no longer JP3.1
- net UP: now also D2.C; no longer JP3.4
Changed lines of the file:
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@@
 <part name="JP2" library="jumper" deviceset="JP1Q" device=""/>
 <part name="JP3" library="jumper" deviceset="JP4Q" device=""/>
+<part name="D1" library="adafruit" deviceset="DIODE" device="DO-1N4148"/>
+<part name="R3" library="rcl" deviceset="R-EU_" device="0204/7" value="10k"/>
+<part name="D2" library="adafruit" deviceset="DIODE" device="DO-1N4148"/>
+<part name="D3" library="adafruit" deviceset="DIODE" device="DO-1N4148"/>
 </parts>
 <sheets>
@@
 <instance part="JP2" gate="A" x="172.72" y="162.56" rot="R90"/>
 <instance part="JP3" gate="B" x="182.88" y="215.9" rot="R180"/>
+<instance part="D1" gate="G$1" x="185.42" y="238.76" smashed="yes" rot="R90">
+<attribute name="NAME" x="184.9374" y="241.3" size="1.778" layer="95" rot="R90"/>
+</instance>
+<instance part="R3" gate="G$1" x="190.5" y="226.06" rot="R180"/>
+<instance part="D2" gate="G$1" x="180.34" y="198.12" smashed="yes" rot="R270">
+<attribute name="NAME" x="180.8226" y="195.58" size="1.778" layer="95" rot="R270"/>
+</instance>
+<instance part="D3" gate="G$1" x="182.88" y="198.12" smashed="yes" rot="R270">
+<attribute name="NAME" x="183.3626" y="195.58" size="1.778" layer="95" rot="R270"/>
+</instance>
 </instances>
 <busses>
@@
 <label x="185.42" y="200.66" size="1.778" layer="95" rot="R270"/>
 </segment>
+<segment>
+<pinref part="R3" gate="G$1" pin="1"/>
+<wire x1="195.58" y1="226.06" x2="195.58" y2="233.68" width="0.1524" layer="91"/>
+<label x="195.58" y="233.68" size="1.778" layer="95"/>
+</segment>
 </net>
 <net name="RIGHT" class="0">
@@
 </segment>
 <segment>
-<pinref part="JP3" gate="B" pin="4"/>
-<wire x1="182.88" y1="208.28" x2="182.88" y2="200.66" width="0.1524" layer="91"/>
-<label x="182.88" y="200.66" size="1.778" layer="95" rot="R270"/>
+<pinref part="D2" gate="G$1" pin="C"/>
+<wire x1="180.34" y1="195.58" x2="180.34" y2="193.04" width="0.1524" layer="91"/>
 </segment>
 </net>
@@
 </segment>
 <segment>
-<pinref part="JP3" gate="B" pin="6"/>
-<wire x1="180.34" y1="208.28" x2="180.34" y2="200.66" width="0.1524" layer="91"/>
-<label x="180.34" y="200.66" size="1.778" layer="95" rot="R270"/>
+<pinref part="D3" gate="G$1" pin="C"/>
+<wire x1="182.88" y1="195.58" x2="182.88" y2="193.04" width="0.1524" layer="91"/>
 </segment>
 </net>
@@
 </segment>
 <segment>
-<pinref part="JP3" gate="B" pin="1"/>
-<wire x1="185.42" y1="223.52" x2="185.42" y2="231.14" width="0.1524" layer="91"/>
-<label x="185.42" y="231.14" size="1.778" layer="95" rot="R270"/>
+<pinref part="D1" gate="G$1" pin="C"/>
+<wire x1="185.42" y1="241.3" x2="185.42" y2="246.38" width="0.1524" layer="91"/>
+<label x="185.42" y="246.38" size="1.778" layer="95"/>
 </segment>
 </net>
@@
 </segment>
 </net>
+<net name="ESP-RX" class="0">
+<segment>
+<pinref part="JP3" gate="B" pin="1"/>
+<wire x1="185.42" y1="223.52" x2="185.42" y2="226.06" width="0.1524" layer="91"/>
+<label x="185.42" y="231.14" size="1.778" layer="95"/>
+<pinref part="D1" gate="G$1" pin="A"/>
+<pinref part="R3" gate="G$1" pin="2"/>
+<wire x1="185.42" y1="226.06" x2="185.42" y2="236.22" width="0.1524" layer="91"/>
+<junction x="185.42" y="226.06"/>
+</segment>
+</net>
+<net name="CH_PD" class="0">
+<segment>
+<pinref part="JP3" gate="B" pin="6"/>
+<wire x1="180.34" y1="208.28" x2="180.34" y2="200.66" width="0.1524" layer="91"/>
+<label x="180.34" y="200.66" size="1.778" layer="95"/>
+<pinref part="D2" gate="G$1" pin="A"/>
+</segment>
+</net>
+<net name="RST" class="0">
+<segment>
+<pinref part="JP3" gate="B" pin="4"/>
+<wire x1="182.88" y1="208.28" x2="182.88" y2="200.66" width="0.1524" layer="91"/>
+<label x="182.88" y="203.2" size="1.778" layer="95"/>
+<pinref part="D3" gate="G$1" pin="A"/>
+</segment>
+</net>
