File: turbo-pcb/turbo.sch (EAGLE design)
At the start: 4 parts

Commit message: update turbo schematic with some notes and add serial server
Other:
- note added: "A4 is fed to pin 2 on the jumper socket, which is N/C"
- note added: "AY1"
- note added: "AY2"
- note added: "Jumper socket"
Changed lines of the file:
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@@
 <sheet>
 <plain>
+<text x="403.86" y="210.82" size="1.778" layer="91">Jumper socket</text>
+<text x="485.14" y="210.82" size="1.778" layer="91">AY1</text>
+<text x="561.34" y="210.82" size="1.778" layer="91">AY2</text>
+<text x="464.82" y="223.52" size="1.778" layer="91">A4 is fed to pin 2 on the jumper socket,
+which is N/C</text>
 </plain>
 <instances>
@@
 </schematic>
 </drawing>
+<compatibility>
+<note version="6.3" minversion="6.2.2" severity="warning">
+Since Version 6.2.2 text objects can contain more than one line,
+which will not be processed correctly with this version.
+</note>
+</compatibility>
 </eagle>
