File: turbo-pcb/turbo-ds.brd (EAGLE design)
At the start: 54 x 48.6 mm, 4 parts

Commit message: clean up repo
Parts:
- moved INPUT 1.27 mm to (116.5, 2.22)
- moved A4 1.27 mm to (94.9, -5.40)
- moved AY1 1.27 mm to (116.5, 8.57)
- moved AY2 1.27 mm to (116.5, 27.6)
Routing:
- net GND: track 90.4 -> 80.6 mm
- net A4: track 85.6 -> 80.6 mm
- net VCC: track 86.6 -> 82.1 mm, vias 0 -> 1
Other:
- board size 54 x 48.6 mm -> 54 x 44.8 mm
